Commit message: inverse kinematics

File: src/scara_robot_description/urdf/gazebo_specifics.xacro (robot description, xacro)
@@ -5,11 +5,11 @@
     </gazebo>
     <gazebo reference="link1">
-        <material>Gazebo/Red</material>
+        <material>Gazebo/Blue</material>
     </gazebo>
     <gazebo reference="link1_h">
-        <material>Gazebo/Green</material>
+        <material>Gazebo/Blue</material>
     </gazebo>
     <gazebo reference="link2">
-        <material>Gazebo/Green</material>
+        <material>Gazebo/Blue</material>
     </gazebo>
     <gazebo reference="link1">
@@ -20,4 +20,8 @@
         <mu1>0.5</mu1>
         <mu2>0.5</mu2>
+        <material>Gazebo/Red</material>
+    </gazebo>
+    <gazebo reference="cyl1">
+        <material>Gazebo/Red</material>
     </gazebo>
     <gazebo reference="link1_h">

File: src/scara_robot_description/urdf/scara_2.urdf.xacro (robot description, xacro)
@@ -47,5 +47,5 @@
     <link name="link1">
         <collision>
-            <origin xyz="0 0 ${a0/2}" rpy="0 0 0"/>
+            <origin xyz="0 0 ${a0}" rpy="0 0 0"/>
             <geometry>
                 <box size="${width} ${width} ${a0*2}"/>
@@ -53,5 +53,5 @@
         </collision>
         <visual>
-            <origin xyz="0 0 ${a0/2}" rpy="0 0 0"/>
+            <origin xyz="0 0 ${a0}" rpy="0 0 0"/>
             <geometry>
                 <box size="${width} ${width} ${a0*2}"/>
@@ -59,10 +59,10 @@
         </visual>
         <inertial>
-            <origin xyz="0 0 ${a0/2}" rpy="0 0 0"/>
+            <origin xyz="0 0 ${a0}" rpy="0 0 0"/>
             <mass value="${mass}"/>
             <inertia
-                ixx="${mass / 12.0 * (width*width + a0*a0)}" ixy="0.0" ixz="0.0"
+                ixx="${mass / 12.0 * (width*width + a0*a0*16)}" ixy="0.0" ixz="0.0"
                 iyy="${mass / 12.0 * (width*width + width*width)}" iyz="0.0"
-                izz="${mass / 12.0 * (width*width + a0*a0)}"/>
+                izz="${mass / 12.0 * (width*width + a0*a0*16)}"/>
         </inertial>
     </link>
@@ -73,21 +73,21 @@
         <axis xyz="0 0 1"/>
         <dynamics damping="0.7"/>
-        <limit lower="0.0" upper="0.5" effort="10" velocity="2"/>
+        <limit lower="0.0" upper="${a0*2}" effort="10" velocity="2"/>
     </joint>
     <link name="cyl0">
         <collision>
-            <origin xyz="0 0 ${a0/2}" rpy="0 0 0"/>
-            <geometry>
-                <cylinder length = "${height1}" radius = "${radius1}"/>
-            </geometry>
-        </collision>
-        <visual>
-            <origin xyz="0 0 ${a0/2}" rpy="0 0 0"/>
-            <geometry>
-                <cylinder length = "${height1}" radius = "${radius1}"/>
-            </geometry>
-        </visual>
-        <inertial>
-            <origin xyz="0 0 0" rpy="0 0 0"/>
+            <origin xyz="0 0 ${height1/2}" rpy="0 0 0"/>
+            <geometry>
+                <cylinder length = "${height1}" radius = "${radius1}"/>
+            </geometry>
+        </collision>
+        <visual>
+            <origin xyz="0 0 ${height1/2}" rpy="0 0 0"/>
+            <geometry>
+                <cylinder length = "${height1}" radius = "${radius1}"/>
+            </geometry>
+        </visual>
+        <inertial>
+            <origin xyz="0 0 ${height1/2}" rpy="0 0 0"/>
             <mass value="2"/>
             <inertia ixx="0.31" ixy="0.0" ixz="0.0" iyy="0.31" iyz="0.0" izz="0.2"/>
@@ -98,5 +98,5 @@
         <parent link="cyl0"/>
         <child link="link1_h"/>
-        <origin xyz="0 0 ${a0/2}" rpy="0 0 0"/>
+        <origin xyz="0 0 ${height1/2}" rpy="0 0 0"/>
         <axis xyz="0 0 1"/>
         <dynamics damping="0.7"/>
